File: alim_DC_DC/Alim_DCDC_12_170/Alim_DCDC_12_170.sch (KiCad schematic (older format))
At the start: 6 parts, among them J1 Conn_01x02_Male, T1 transformer_flyback_4P_1S, U1 LT3757AEMSE

Commit message: schéma fini
Parts:
- removed R? (x2): R, symbol Device:R
- added C1, C2, C3, C4, C5, C6, C7: C, symbol Device:C
- added D1: D, symbol Device:D
- added J2: Conn_01x02_Female, symbol Connector:Conn_01x02_Female
- added R1, R2, R3, R4, R5, R6, R7, R8, R9: R, symbol Device:R
- T1: footprint (none) -> Transformer_SMD:Transformer_Coilcraft_DA2032_AL
- gave numbers to parts that had none: 1
Connections:
- net GND: now also J1.2 (Pin_2), T1.1, C1.2, C2.2, C3.2, C4.2, C5.2, C6.2, C7.2, J2.2 (Pin_2), R1.2, R2.2, R6.2, R9.2
- net HT: now also J2.1 (Pin_1)
- net VCC: now also J1.1 (Pin_1), T1.10, T1.7, T1.8, T1.9, U1.8 (INTVCC), C7.1, R3.1
- net at U1.1 (VC): now also C2.1, R4.1
- net at U1.2 (FBX): now also R8.2, R9.1
- net at U1.3 (SS): now also C1.1
- net at U1.4 (RT): now also R2.1
- net at U1.6 (SENSE): now also C4.1, R5.1
- net at U1.7 (GATE): now also Q1.1 (G)
- net at U1.9 (~SHDN~/UVLO): now also R1.1, R3.2
- net at T1.12: now also D1.2 (A)
- net at T1.3: now also Q1.2 (D), Q1.4 (D), T1.4, T1.5, T1.6
- net at Q1.3 (S): now also R5.2, R6.1
- new net: C3.1, R4.2
- new net: C5.1, C6.1, D1.1 (K), R7.1
- new net: R7.2, R8.1
Other:
- moved on the sheet: Q1, T1

Commit message: some new names and values pt. 1
Parts:
- added C2, C3, C4, C5: C, symbol Device:C
- C1: value C -> 100n
- C10: renamed from C2; value C -> 100p
- C9: renamed from C3; value C -> 22n
- R1: renamed from R2; value R -> 140k
- R6: renamed from R4; value R -> 6.8k
- R8: renamed from R3; value R -> 100k
- R9: renamed from R1; value R -> 4.3k
- renumbered C7 to C12, C4 to C?, C5 to C?, C6 to C?, D1 to D?, J1 to J?, J2 to J?, Q1 to Q?, R5 to R?, R6 to R?, R7 to R?, R8 to R?, R9 to R?, T1 to T?, U1 to U?
Connections:
- net GND: now also C2.2, C3.2, C4.2, C5.2
- net VCC: now also C2.1, C3.1, C4.1, C5.1
Other:
- moved on the sheet: C9, R6
